File: TwomesSensor/TwomesSensor.kicad_pcb (KiCad board)
At the start: 2 copper layers, 73 x 77 mm, 50 parts, among them J1 Female header, J2 Molex PicoFlex 90814, J3 Molex PicoFlex 90814, J4 Molex PicoFlex 90814, J5 Molex PicoFlex 90814, Q1 PMV48XP,215, Q2 PMV48XP,215, SW1 SW_Push, SW2 SW_Push, SW3 SW_Push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

Commit message: Update CO2 sensor footprint
Other:
- board text added: "Twomes Sensor V2.0 June 2021"
- board text added: "Version 2.0 Designed By Sjors Smit June 2021"
- board text removed: "Twomes Sensor V2.0 April 2021"
- board text removed: "Version 2.0 Designed By Sjors Smit April 2021"
